File: DevBrix Custom Design Block.kicad_blocks/Buck +12V collections.kicad_block/Buck +12V collections.kicad_sch (KiCad schematic)
At the start: 13 parts, among them U7 LMR51450SDRRR

Commit message: add more library
Parts:
- C1: renamed from C36; footprint custom_lib:C_0805_2012Metric -> Capacitor_SMD:C_0805_2012Metric; symbol custom_lib:C_Small -> Device:C_Small
- C2: renamed from C37; footprint custom_lib:C_0402_1005Metric -> Capacitor_SMD:C_0402_1005Metric; symbol custom_lib:C_Small -> Device:C_Small
- C3: renamed from C38; footprint custom_lib:C_0402_1005Metric -> Capacitor_SMD:C_0402_1005Metric; symbol custom_lib:C_Small -> Device:C_Small; LCSC (none) -> C1525; Rating (none) -> 16V
- C4: renamed from C39; footprint custom_lib:C_0805_2012Metric -> Capacitor_SMD:C_0603_1608Metric; symbol custom_lib:C_Small -> Device:C_Small; LCSC C2932476 -> C96446
- C5: renamed from C40; footprint custom_lib:C_0805_2012Metric -> Capacitor_SMD:C_0603_1608Metric; symbol custom_lib:C_Small -> Device:C_Small; LCSC C2932476 -> C96446
- C6: renamed from C41; footprint custom_lib:C_0402_1005Metric -> Capacitor_SMD:C_0402_1005Metric; symbol custom_lib:C_Small -> Device:C_Small; LCSC (none) -> C100072
- C7: renamed from C42; footprint custom_lib:C_0402_1005Metric -> Capacitor_SMD:C_0402_1005Metric; symbol custom_lib:C_Small -> Device:C_Small; LCSC (none) -> C70465
- L1: renamed from L3; footprint custom_lib:L_Coilcraft_XxL4020 -> Inductor_SMD:L_Changjiang_FXL0640; symbol custom_lib:L_Small -> Device:L_Small; LCSC (none) -> C53426759; Rating (none) -> 5A
- R1: renamed from R18; symbol custom_lib:R_Small -> Device:R_Small; LCSC (none) -> C25543
- R2: renamed from R19; footprint custom_lib:R_0402_1005Metric -> Resistor_SMD:R_0402_1005Metric; symbol custom_lib:R_Small -> Device:R_Small; LCSC (none) -> C270658
- R3: renamed from R20; symbol custom_lib:R_Small -> Device:R_Small; LCSC (none) -> C21376
- R4: renamed from R21; footprint custom_lib:R_0402_1005Metric -> Resistor_SMD:R_0402_1005Metric; symbol custom_lib:R_Small -> Device:R_Small; LCSC (none) -> C270586
- U1: renamed from U7; footprint Package_SON:WSON-12-1EP_3x3mm_P0.5mm_EP1.5x2.5mm -> DevBriX Custom Library:WSON-12-DRR0012G; Check (none) -> OK
Connections:
- net ~{SYS_RESET} renamed EN
Other:
- moved on the sheet: C1, C2, C3, C4, C5, C6, C7, L1, R1, R2, R3, R4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
