File: DevBrix Custom Design Block.kicad_blocks/USB PD STUSB4500.kicad_block/USB PD STUSB4500.kicad_sch (KiCad schematic)
At the start: 25 parts, among them J1 GT-USB-7002C, Q1 AO4805, U2 STUSB4500QTR

Commit message: add more library
Parts:
- C1: footprint custom_lib:C_0805_2012Metric -> Capacitor_SMD:C_0805_2012Metric; symbol custom_lib:C_Small -> Device:C_Small
- C2, C5, C6: footprint custom_lib:C_0402_1005Metric -> Capacitor_SMD:C_0402_1005Metric; symbol custom_lib:C_Small -> Device:C_Small
- C3, C4: footprint custom_lib:C_0603_1608Metric -> Capacitor_SMD:C_0603_1608Metric; symbol custom_lib:C_Small -> Device:C_Small
- R1, R2, R3, R4, R5, R6, R7: footprint custom_lib:R_0402_1005Metric -> Resistor_SMD:R_0402_1005Metric; symbol custom_lib:R_Small -> Device:R_Small
- TP1, TP2, TP3, TP4, TP5: footprint custom_lib:TestPoint_Pad_D1.0mm -> TestPoint:TestPoint_Pad_D1.0mm; symbol custom_lib:TestPoint -> Connector:TestPoint
- U1: renamed from U?; LCSC (none) -> C2935152; LCSC Part C2935152 -> (none)
Other:
- moved on the sheet: C1, C2, C3, C4, C5, C6, D1, D2, D3, J1, Q1A, Q1B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
