File: DevBrix Custom Template/Generic Project/Generic Project.kicad_pcb (KiCad board)
At the start: 10 copper layers, 21.3 x 70 mm, 247 parts, among them IC1 MP2143DJ-LF-Z, J1 Conn_01x19_Pin, J11 54548-2271, J12 Conn_01x08_Pin, J13 Conn_01x08_Pin, J2 Conn_01x19_Pin, J3 HDMI_D_1.4, J5 USB_C, J6 RJ-45, J7 B2B-PH-SM4-TB (LF)(SN), J8 MEM2085-00-115-00-A, J9 U.FL, Q1 PMPB12R5EPX, SW1 BUTTON, U1 USBLC6-2SC6, U10 RTL8211E-VB-CG, U11 MAX17048G+T10, U12 ADV7535BCBZ-RL7, U13 TPD4E02B04DQA, U14 TLV75733PDRV, U15 TPS2116DRL, U16 TPS61033DRLR, U17 STM32L011E4Yx, U18 TPS2116DRL, U2 TPD4E02B04DQA, U3 LBES5PL2EL-923, U4 APS6404L-3SQR-ZR, U5 SGTL5000XNLA3, U6 TPS62A02DRL, U7 W25Q256JVPIQ, U8 MIMXRT1176DVMAB, U9 BQ24040DSQR, Y1 24MHz, Y2 32.768KHz, Y3 25MHz

Commit message: add new library
Parts:
- removed AE1: Antenna_Chip, M830520:M830520
- removed C1, C118, C13, C15, C16, C17, C20, C22, C25, C27, C28, C30, C31, C38, C39, C4, C42, C60, C64, C75, C78, C84, C87: 1uF 10V, Passive:C_0201
- removed C10: 22uF 10V, Capacitor_SMD:C_0603_1608Metric
- removed C100, C2, C29, C34, C35, C48, C62, C63, C65, C66, C67, C70, C89, C98: 4.7uF 6.3V, Passive:C_0201
- removed C101, C102, C103, C104, C11, C110, C115, C116, C119, C12, C120, C123, C124, C126, C127, C128, C26, C32, C51, C57, C59, C61, C73, C74, C80, C82, C85, C86, C88, C9, C92, C93, C94, C95, C97, C99: 0.1uF 10V, Passive:C_0201
- removed C107: 27pF 50V, Passive:C_0201
- removed C108, C109: 22pF 50V, Passive:C_0201
- removed C113, C114, C117, C121, C122, C125: 10uF 6.3V, Capacitor_SMD:C_0402_1005Metric
- removed C14, C21, C41, C44, C5, C68, C8: 0.22uF 6.3V, Passive:C_0201
- removed C18, C19, C3, C33, C40, C56, C6, C90: 10uF 10V, Capacitor_SMD:C_0402_1005Metric
- removed C23, C24, C36, C37, C43, C47, C52, C53, C54, C69, C72, C76, C77, C81: 2.2uF 6.3V, Passive:C_0201
- removed C45, C46: 18pF 50V, Passive:C_0201
- removed C49, C50: 10pF, Passive:C_0201
- removed C55, C58, C7, C83, C91, C96: 22uF 6.3V, Capacitor_SMD:C_0603_1608Metric
- removed C71: 10pF 50V, Passive:C_0201
- removed C79: 1nF 25V, Passive:C_0201
- removed D1: ESD5Z5.0T1G, Diode_SMD:D_SOD-523
- removed D2, D5: 18-225/R6G6C-A01/3T, 18-225_R6G6C-A01_3T:18-225_R6G6C-A01_3T
- removed D3: TX1812LB, TX1812LB:TX1812LB
- removed D4: NSR20F30NXT5G, NSR20F30NXT5G:NSR20F30NXT5G
- removed F1: 500mA, Fuse:Fuse_0402_1005Metric
- removed H1, H2, H3, H4: MountingHole, MountingHole:MountingHole_2.5mm
- removed IC1: MP2143DJ-LF-Z, Package_TO_SOT_SMD:TSOT-23-8
- removed J1, J2: Conn_01x19_Pin, Connector_PinHeader_2.54mm:PinHeader_1x19_P2.54mm_Vertical
- removed J11: 54548-2271, 54548-2271:545482271
- removed J12, J13: Conn_01x08_Pin, Connector_PinHeader_2.54mm:PinHeader_1x08_P2.54mm_Vertical
- removed J3: HDMI_D_1.4, Connector_Video:HDMI_Micro-D_Molex_46765-2xxx
- removed J5: USB_C, Connector_USB:USB_C_Receptacle_HRO_TYPE-C-31-M-12
- removed J6: RJ-45, Connector_PinHeader_1.27mm:PinHeader_2x06_P1.27mm_Vertical
- removed J7: B2B-PH-SM4-TB (LF)(SN), Connector_JST:JST_PH_B2B-PH-SM4-TB_1x02-1MP_P2.00mm_Vertical
- removed J8: MEM2085-00-115-00-A, MEM2085-00-115-00-A:MEM2085-00-115-00-A
- removed J9: U.FL, Connector_Coaxial:U.FL_Hirose_U.FL-R-SMT-1_Vertical
- removed L1, L10, L2, L3, L5, L9: 120Ω, Inductor_SMD:L_0402_1005Metric
- removed L11: 0.47uH, Inductor_SMD:L_Coilcraft_XAL4020-XXX
- removed L12: 2.2uH, Inductor_SMD:L_Murata_DFE201610P
- removed L4: 4.7uH, Inductor_SMD:L_Sunlord_SWPA4020S
- removed L6: 1uH, Inductor_SMD:L_Murata_DFE201610P
- removed L8: 1uH, Inductor_SMD:L_Sunlord_SWPA4020S
- removed MIC1: IMP23ABSUTR, IMP23ABSUTR:IMP23ABSUTR
- removed Q1: PMPB12R5EPX, PMPB12R5EPX:PMPB12R5EPX
- removed R1, R14, R19, R22, R25, R6: 10K, Passive:R_0201
- removed R10, R29, R9: 0R, Passive:R_0201
- removed R11, R12: 5.1K, Passive:R_0201
- removed R13, R15, R20, R21, R42: 1.5K, Passive:R_0201
- removed R16: 1K, Passive:R_0201
- removed R17: 2K, Passive:R_0201
- removed R18, R32, R33: 470K, Passive:R_0201
- removed R2, R26, R31, R60, R61, R62, R63, R64: 100K, Passive:R_0201
- removed R23, R24, R34, R48, R49, R50, R51, R52, R53, R54, R55: 22R, Passive:R_0201
- removed R27: 180K, Passive:R_0201
- removed R28: 40.2K, Passive:R_0201
- removed R3: 2k, Passive:C_0201
- removed R30: 30K, Passive:R_0201
- removed R35, R37, R38, R39, R4, R40, R41, R43, R44, R45, R5, R58: 4.7K, Passive:R_0201
- removed R36: 2.49K, Passive:R_0201
- removed R46, R47: 390R, Passive:R_0201
- removed R56, R57: 1k, Passive:C_0201
- removed R59: 200K, Passive:R_0201
- removed R7: 931K, Passive:R_0201
- removed R8: 127K, Passive:R_0201
- removed S1: TPD3S014TDBVRQ1, TPD3S014TDBVRQ1:TPD3S014TDBVRQ1
- removed SW1: BUTTON, TS-1185-B-A-B-A:TS-1185-B-A-B-A
- removed U10: RTL8211E-VB-CG, RTL8211E-VB-CG:RTL8211E-VB-CG
- removed U11: MAX17048G+T10, Package_DFN_QFN:TDFN-8-1EP_2x2mm_P0.5mm_EP0.8x1.2mm
- removed U12: ADV7535BCBZ-RL7, ADV7535BCBZ-RL7:ADV7535BCBZ-RL7
- removed U13, U2: TPD4E02B04DQA, Package_SON:USON-10_2.5x1.0mm_P0.5mm
- removed U14: TLV75733PDRV, Package_SON:WSON-6-1EP_2x2mm_P0.65mm_EP1x1.6mm
- removed U15, U18: TPS2116DRL, Package_TO_SOT_SMD:SOT-583-8
- removed U16: TPS61033DRLR, Package_TO_SOT_SMD:SOT-583-8
- removed U17: STM32L011E4Yx, Package_CSP:ST_WLCSP-25_Die457
- removed U3: LBES5PL2EL-923, LBES5PL2EL-923:LBES5PL2EL923
- removed U4: APS6404L-3SQR-ZR, APS6404L-3SQR-ZR:APS6404L-3SQR-ZR
- removed U5: SGTL5000XNLA3, Package_DFN_QFN:QFN-20-1EP_3x3mm_P0.4mm_EP1.65x1.65mm
- removed U6: TPS62A02DRL, Package_TO_SOT_SMD:SOT-563
- removed U7: W25Q256JVPIQ, W25Q128JVPIQ:W25Q128JVPIQ
- removed U8: MIMXRT1176DVMAB, MIMXRT1176DVMAA:MIMXRT1176DVMAA
- removed U9: BQ24040DSQR, Package_DFN_QFN:Texas_DSQ0010A_WSON-10-1EP_2x2mm_P0.4mm_EP0.9x1.5mm
- removed Y1: 24MHz, Crystal:Crystal_SMD_2016-4Pin_2.0x1.6mm
- removed Y2: 32.768KHz, Crystal:Crystal_SMD_3215-2Pin_3.2x1.5mm
- removed Y3: 25MHz, Crystal:Crystal_SMD_2016-4Pin_2.0x1.6mm
- U1: value USBLC6-2SC6 -> W25Q16JVSS; footprint Package_TO_SOT_SMD:SOT-23-6 -> Package_SO:SOIC-8_5.3x5.3mm_P1.27mm; moved to F.Cu
- moved U1 73.8 mm to (135.9, 104.7), turned to 0 degrees
Connections:
- U1 pad 1: Net-(J5-D+-PadA6) -> unconnected-(U1-~{CS}-Pad1)
- U1 pad 2: GND -> unconnected-(U1-DO/IO_{1}-Pad2)
- U1 pad 3: Net-(J5-D--PadA7) -> unconnected-(U1-~{WP}/IO_{2}-Pad3)
- U1 pad 4: Net-(R9-Pad1) -> unconnected-(U1-GND-Pad4)
- U1 pad 5: VBUS -> unconnected-(U1-DI/IO_{0}-Pad5)
- U1 pad 6: Net-(R10-Pad2) -> unconnected-(U1-CLK-Pad6)
Routing:
- net +3V3: track 84.7 -> 0.00 mm, vias 38 -> 0
- net I2C1_SDA: track 67.4 -> 0.00 mm, vias 11 -> 0
- net I2C1_SCL: track 67.3 -> 0.00 mm, vias 11 -> 0
- net GND: track 44.0 -> 0.00 mm, vias 61 -> 0
- net SD_SDIO2_D1: track 41.7 -> 0.00 mm, vias 6 -> 0
- net SD_SDIO2_D0: track 41.6 -> 0.00 mm, vias 6 -> 0
- net SD_SDIO2_D2: track 41.1 -> 0.00 mm, vias 6 -> 0
- net SD_SDIO2_D3: track 41.1 -> 0.00 mm, vias 6 -> 0
- net SD_SDIO2_CMD: track 41.0 -> 0.00 mm, vias 6 -> 0
- net SD_SDIO2_CLK: track 41.0 -> 0.00 mm, vias 6 -> 0
- net CSI_DN0: track 39.3 -> 0.00 mm, vias 5 -> 0
- net CSI_DP0: track 39.2 -> 0.00 mm, vias 5 -> 0
- net CSI_DN1: track 36.8 -> 0.00 mm, vias 5 -> 0
- net CSI_DP1: track 36.8 -> 0.00 mm, vias 5 -> 0
- net +5V: track 34.8 -> 0.00 mm
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- removed copper zone on In5.Cu, net +1V8
- removed copper zone on In5.Cu, net +3V3
- removed copper zone on In5.Cu, net +5V
- removed copper zone on In5.Cu, net /Ethernet PHY/+1V0_ETH
- removed copper zone on F.Cu, net /SoC Power Pins/VDD_SOC_IN
- removed copper zone on In5.Cu, net /SoC Power Pins/VDD_SOC_IN
- removed copper zone on B.Cu, net GND
- removed copper zone on F.Cu, net GND
- removed copper zone on In1.Cu, net GND
- removed copper zone on In2.Cu, net GND
- removed copper zone on In3.Cu, net GND
- removed copper zone on In4.Cu, net GND
- removed copper zone on In6.Cu, net GND
- removed copper zone on In7.Cu, net GND
- removed copper zone on In8.Cu, net GND
- removed copper zone on In5.Cu, net Net-(U8B-ADC_VREFH)
- removed copper zone on In5.Cu, net VCC
- removed copper zone on In5.Cu, net VDC
- removed copper zone on In5.Cu, net VDDA_1V0
Other:
- board outline removed
- copper layers 10 -> 2
