File: DevBrix Custom Template/Generic Project/Generic Project.kicad_sch (KiCad schematic)
At the start: 0 parts

Commit message: add new library
Changed lines of the file:
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@@
 		(margins 0.9525 0.9525 0.9525 0.9525)
 		(stroke
-			(width 0.254)
+			(width 0.381)
 			(type solid)
 		)
